File: pcb/dev_board.kicad_sch (KiCad schematic)
At the start: 38 parts, among them J1 Conn_02x13_Odd_Even, J2 Conn_02x13_Odd_Even, J4 Conn_01x05, SW1 SW_DIP_x03, SW2 Start, U1 XS-LPC-01, U2 MCP3202, U3 TLV75530PDBV, U6 TLV74311

Commit message: V0.2 schem, bom, pcb. Ready to route
Parts:
- removed R15: 1R 3W 0.1%, Resistor_SMD:R_2512_6332Metric, symbol Device:R
- J4: footprint Connector_PinHeader_2.54mm:PinHeader_1x05_P2.54mm_Vertical_SMD_Pin1Left -> Connector_JST:CONN_B5B-ZR-SM4-TF_JST; DPN SAM10797-ND -> 455-1684-1-ND
- R8: value 18R6 -> 47; DPN 311-18.2HRCT-ND -> 541-47.0HCT-ND
- U3: value TLV75530PDBV -> NCP114ASN280T1G; DPN 576-4905-1-ND -> NCP114ASN280T1GOSCT-ND
Connections:
- net CT1: now also R8.2; no longer R8.1
- net CT2: now also R8.1; no longer R8.2
Other:
- note added: "Connector / Protection"
- note added: "Voltage Regs"
- note removed: "Connector"
- moved on the sheet: C1, C10, C3, C4, C5, C6, C7, C8, C9, D1, D2, D3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
