File: pcb/dev_board.kicad_sch (KiCad schematic)
At the start: 39 parts, among them J1 Conn_02x13_Odd_Even, J2 Conn_02x13_Odd_Even, J4 Conn_01x05, SW1 SW_DIP_x03, SW2 Start, U1 XS-LPC-01, U2 MCP3202, U3 NCP114ASN280T1G, U6 TLV74311

Commit message: PCB Tapeout v0.5 LPC_DB development board, schematic, bom, datasheets updated.
Parts:
- added TP1: GND, TestPoint:TestPoint_Keystone_5000-5004_Miniature, symbol Connector:TestPoint
Connections:
- net +3V0: now also R10.3; no longer R10.1
- net CT2: now also R10.1; no longer R10.3
- net GND: now also TP1.1
Other:
- note added: "mid 1.5v"
Changed lines of the file:
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@@
     (title "XS-LPC-DB Development Board")
     (date "2026-07-10")
-    (rev "v0.3")
+    (rev "v0.5")
     (company "Eric Pearson, XYZZY Semiconductor")
   )
@@
     (effects (font (size 6 6)) (justify left bottom))
   )
+  (text "mid 1.5v" (at 66.675 178.435 0)
+    (effects (font (size 1.27 1.27)) (justify left bottom))
+  )
   (label "fault_led" (at 87.63 111.125 0) (fields_autoplaced)
     (effects (font (size 1.27 1.27)) (justify left bottom))
@@
     (effects (font (size 1.27 1.27)) (justify right bottom))
   )
-  (label "mid1v5" (at 56.515 178.435 0) (fields_autoplaced)
-    (effects (font (size 1.27 1.27)) (justify left bottom))
-  )
   (label "timeout" (at 77.47 118.745 180) (fields_autoplaced)
     (effects (font (size 1.27 1.27)) (justify right bottom))
@@
     )
   )
-  (symbol (lib_id "Device:R_Potentiometer_US") (at 64.77 172.085 0) (unit 1)
+  (symbol (lib_id "Device:R_Potentiometer_US") (at 64.77 172.085 0) (mirror x) (unit 1)
     (in_bom yes) (on_board yes) (dnp no)
-    (property "Reference" "R10" (at 62.23 170.18 0)
+    (property "Reference" "R10" (at 62.23 173.99 0)
       (effects (font (size 1.27 1.27)) (justify right))
     )
-    (property "Value" "1K" (at 61.595 173.355 0)
+    (property "Value" "1K" (at 61.595 170.815 0)
       (effects (font (size 1.27 1.27)) (justify right))
     )
@@
     )
   )
+  (symbol (lib_id "power:GND") (at 236.22 144.78 0) (unit 1)
+    (in_bom yes) (on_board yes) (dnp no) (fields_autoplaced)
+    (property "Reference" "#PWR018" (at 236.22 151.13 0)
+      (effects (font (size 1.27 1.27)) hide)
+    )
+    (property "Value" "GND" (at 236.22 149.86 0)
+      (effects (font (size 1.27 1.27)))
+    )
+    (property "Footprint" "" (at 236.22 144.78 0)
+      (effects (font (size 1.27 1.27)) hide)
+    )
+    (property "Datasheet" "" (at 236.22 144.78 0)
+      (effects (font (size 1.27 1.27)) hide)
+    )
+    (pin "1")
+    (instances
+      (project "dev_board"
+        (path "/91657278-176c-4c3c-b7c8-7fab77e89520"
+          (reference "#PWR018") (unit 1)
+        )
+      )
+    )
+  )
   (symbol (lib_id "Device:C_Small") (at 92.075 185.42 0) (unit 1)
     (in_bom yes) (on_board yes) (dnp no) (fields_autoplaced)
@@
         )
       )
+    )
+  )
+  (symbol (lib_id "Connector:TestPoint") (at 236.22 144.78 0) (unit 1)
+    (in_bom yes) (on_board yes) (dnp no)
+    (property "Reference" "TP1" (at 234.95 139.7 0)
+      (effects (font (size 1.27 1.27)) (justify left))
+    )
+    (property "Value" "GND" (at 238.76 143.383 0)
+      (effects (font (size 1.27 1.27)) (justify left))
+    )
+    (property "Footprint" "TestPoint:TestPoint_Keystone_5000-5004_Miniature" (at 241.3 144.78 0)
+      (effects (font (size 1.27 1.27)) hide)
+    )
+    (property "Datasheet" "https://www.digikey.ca/en/products/detail/keystone-electronics/1037/315153" (at 241.3 144.78 0)
+      (effects (font (size 1.27 1.27)) hide)
+    )
+    (property "OK" "" (at 236.22 144.78 0)
+      (effects (font (size 1.27 1.27)) hide)
+    )
+    (property "DPN" "36-1037-ND" (at 236.22 144.78 0)
+      (effects (font (size 1.27 1.27)) hide)
+    )
+    (pin "1")
+    (instances
+      (project "dev_board"
+        (path "/91657278-176c-4c3c-b7c8-7fab77e89520"
+          (reference "TP1") (unit 1)
+        )
+      )
